Commit message: Line Following Complete

File: src/description/Depth_camera.xacro (robot description, xacro)
@@ -1,24 +1,24 @@
 <?xml version="1.0"?>
 <robot xmlns:xacro="http://www.ros.org/wiki/xacro" >
-    <joint name="camera_joint" type="fixed">
-        <parent link="chassis"/>
-        <child link="camera_link"/>
-        <origin xyz="0.305 0 0.08" rpy="0 0 0"/>
+    <joint name="Depth_camera_joint" type="fixed">
+        <parent link="base_link"/>
+        <child link="Depth_camera_link"/>
+        <origin xyz="0.31 0 0.085" rpy="0 0 0"/>
     </joint>
-    <link name="camera_link">
+    <link name="Depth_camera_link">
         <visual>
             <geometry>
-                <box size="0.010 0.03 0.03"/>
+                <box size="0.04 0.04 0.07"/>
             </geometry>
             <material name="red"/>
         </visual>
     </link>
-    <joint name="camera_optical_joint" type="fixed">
-        <parent link="camera_link"/>
-        <child link="camera_link_optical"/>
-        <origin xyz="0 0 0" rpy="${-pi/2} 0 ${-pi/2}"/>
+    <joint name="Depth_camera_optical_joint" type="fixed">
+        <parent link="Depth_camera_link"/>
+        <child link="Depth_camera_link_optical"/>
+        <origin xyz="0 0 -0.035" rpy="${-pi/2} 0 ${-pi/2}"/>
     </joint>
-    <link name="camera_link_optical"></link>
-    <gazebo reference="camera_link">
+    <link name="Depth_camera_link_optical"></link>
+    <gazebo reference="Depth_camera_link">
         <material>Gazebo/Red</material>
         <sensor name="camera" type="depth">
@@ -38,6 +38,6 @@
                 </clip>
             </camera>
-            <plugin name="camera_controller" filename="libgazebo_ros_camera.so">
-                <frame_name>camera_link_optical</frame_name>
+            <plugin name="Depth_camera_controller" filename="libgazebo_ros_camera.so">
+                <frame_name>Depth_camera_link_optical</frame_name>
             </plugin>
         </sensor>

File: src/description/camera.xacro (robot description, xacro)
@@ -1,9 +1,4 @@
 <?xml version="1.0"?>
 <robot xmlns:xacro="http://www.ros.org/wiki/xacro" >
-    <joint name="camera_joint" type="fixed">
-        <parent link="chassis"/>
-        <child link="camera_link"/>
-        <origin xyz="0.305 0 0.08" rpy="0 0 0"/>
-    </joint>
     <link name="camera_link">
         <visual>
@@ -14,4 +9,10 @@
         </visual>
     </link>
+    <joint name="camera_joint" type="fixed">
+        <parent link="camera_platform_link"/>
+        <child link="camera_link"/>
+        <origin xyz="0.235 0 -0.02" rpy="0 ${pi/2} 0"/>
+    </joint>
+    <link name="camera_link_optical"></link>
     <joint name="camera_optical_joint" type="fixed">
         <parent link="camera_link"/>
@@ -19,5 +20,4 @@
         <origin xyz="0 0 0" rpy="${-pi/2} 0 ${-pi/2}"/>
     </joint>
-    <link name="camera_link_optical"></link>
     <gazebo reference="camera_link">
         <material>Gazebo/Red</material>

File: src/description/gazebo_control.xacro (robot description, xacro)
@@ -4,8 +4,8 @@
         <plugin name="diff_drive" filename="libgazebo_ros_diff_drive.so">
             <!-- Wheel Information -->
-            <left_joint>left_wheel_joint</left_joint>
-            <right_joint>right_wheel_joint</right_joint>
+            <left_joint>back_left_wheel_joint</left_joint>
+            <right_joint>back_right_wheel_joint</right_joint>
             <wheel_separation>0.35</wheel_separation>
-            <wheel_diameter>0.1</wheel_diameter>
+            <wheel_diameter>0.14</wheel_diameter>
             <!-- Limits -->
             <max_wheel_torque>200</max_wheel_torque>
@@ -13,5 +13,5 @@
             <!-- Output -->
             <odometry_frame>odom</odometry_frame>
-            <robot_base_frame>base_link</robot_base_frame>
+            <robot_base_frame>back_base_link</robot_base_frame>
             <publish_odom>true</publish_odom>
             <publish_odom_tf>true</publish_odom_tf>

File: src/description/lidar.xacro (robot description, xacro)
@@ -1,8 +1,29 @@
 <?xml version="1.0"?>
 <robot xmlns:xacro="http://www.ros.org/wiki/xacro">
+    <link name="platform">
+        <visual>
+            <geometry>
+                <box size="0.15 0.3 0.075"/>
+            </geometry>
+            <material name="white"/>
+        </visual>
+        <collision>
+            <geometry>
+                <box size="0.15 0.15 0.075"/>
+            </geometry>
+        </collision>
+        <xacro:inertial_box mass="0.5" x="0.3" y="0.3" z="0.15">
+            <origin xyz="0 0 0" rpy="0 0 0"/>
+        </xacro:inertial_box>
+    </link>
+    <joint name="laser_platform" type="fixed">
+        <parent link="base_link"/>
+        <child link="platform"/>
+        <origin xyz="0 0 0.112" rpy="0 0 0"/>
+    </joint>
     <joint name="laser_joint" type="fixed">
-        <parent link="chassis"/>
+        <parent link="platform"/>
         <child link="laser_frame"/>
-        <origin xyz="0.1 0 0.175" rpy="0 0 0"/>
+        <origin xyz="0 0 0.057" rpy="0 0 0"/>
     </joint>
     <link name="laser_frame">

File: src/description/robot.urdf.xacro (robot description, xacro)
@@ -1,7 +1,8 @@
 <?xml version="1.0"?>
-<robot xmlns:xacro="http://www.ros.org/wiki/xacro"  name="robot">
+<robot xmlns:xacro="http://www.ros.org/wiki/xacro"  name="nav_robot">
     <xacro:include filename="robot_core.xacro"/>
-    <!-- <xacro:include filename="gazebo_control.xacro"/> -->
-    <xacro:include filename="ros2_control.xacro"/>
+    <!-- <xacro:include filename="test.xacro"/> -->
+    <xacro:include filename="gazebo_control.xacro"/>
+    <!-- <xacro:include filename="ros2_control_back.xacro"/>  -->
     <xacro:include filename="lidar.xacro"/>
     <xacro:include filename="camera.xacro"/>

File: src/description/robot_core.xacro (robot description, xacro)
@@ -1,5 +1,6 @@
 <?xml version="1.0"?>
 <robot xmlns:xacro="http://www.ros.org/wiki/xacro">
-    <xacro:include filename="inertial_macros.xacro"/>
+    <xacro:include filename="$(find navigation_bot)/description/inertial_macros.xacro"/>
+<!--================================================================ COLOURS ==================================================================================================== -->
     <material name="white">
         <color rgba="1 1 1 1"/>
@@ -17,16 +18,7 @@
         <color rgba="0 0 0 1"/>
     </material>
-    <!-- BASE LINK -->
-    <link name="base_link">
-    </link>
-    <!-- CHASSIS LINK -->
-    <joint name="chassis_joint" type="fixed">
-        <parent link="base_link"/>
-        <child link="chassis"/>
-        <origin xyz="-0.1 0 0"/>
-    </joint>
-    <link name="chassis">
-        <visual>
-        <origin xyz="0.15 0 0.075"/>
+<!--================================================================ LINKS ====================================================================================================== -->
+    <link name="origin"> <!-- base_link LINK -->
+        <visual>
             <geometry>
                 <box size="0.3 0.3 0.15"/>
@@ -35,5 +27,4 @@
         </visual>
         <collision>
-        <origin xyz="0.15 0 0.075"/>
             <geometry>
                 <box size="0.3 0.3 0.15"/>
@@ -41,88 +32,356 @@
         </collision>
         <xacro:inertial_box mass="0.5" x="0.3" y="0.3" z="0.15">
-            <origin xyz="0.15 0 0.075" rpy="0 0 0"/>
-        </xacro:inertial_box>
-    </link>
-    <gazebo reference="chassis">
-        <material>Gazebo/White</material>
-    </gazebo>
-    <!-- LEFT WHEEL LINK -->
-    <joint name="left_wheel_joint" type="continuous">
-        <parent link="base_link"/>
-        <child link="left_wheel"/>
-        <origin xyz="0 0.175 0" rpy="-${pi/2} 0 0"/>
-        <axis xyz ="0 0 1"/>
-    </joint>
-    <link name="left_wheel">
-        <visual>
-            <geometry>
-                <cylinder radius= "0.05" length="0.04"/>
-            </geometry>
-            <material name="blue"/>
-        </visual>
-        <collision>
-            <geometry>
-                <cylinder radius= "0.05" length="0.04"/>
-            </geometry>
-        </collision>
-        <xacro:inertial_cylinder mass="0.1" length="0.04" radius="0.05">
+            <origin xyz="0 0 0" rpy="0 0 0"/>
+        </xacro:inertial_box>
+    </link>
+    <link name="base_link"> <!-- base_link LINK -->
+    </link>
+    <link name="Back_base_link">
+        <visual>
+            <origin xyz="0 0 0" rpy="${pi/2} 0 0"/>
+            <axis xyz ="0 0 1"/>
+            <geometry>
+                <cylinder radius= "0.01" length="0.4"/>
+            </geometry>
+            <material name="blue"/>
+        </visual>
+    </link>
+    <link name="Front_base_link">
+        <visual>
+            <origin xyz="0 0 0" rpy="${pi/2} 0 0"/>
+            <axis xyz ="0 0 1"/>
+            <geometry>
+                <cylinder radius= "0.01" length="0.4"/>
+            </geometry>
+            <material name="blue"/>
+        </visual>
+    </link>
+    <link name="LeftFront_wheel_support">
+        <visual>
+            <geometry>
+                <box size="0.3 0.15 0.03"/>
+            </geometry>
+            <material name="white"/>
+        </visual>
+        <collision>
+            <geometry>
+                <box size="0.3 0.15 0.03"/>
+            </geometry>
+        </collision>
+        <xacro:inertial_box mass="0.32" x="0.3" y="0.3" z="0.15">
+            <origin xyz="0 0 0" rpy="0 0 0"/>
+        </xacro:inertial_box>
+    </link>
+    <link name="RightFront_wheel_support">
+        <visual>
+            <geometry>
+                <box size="0.3 0.15 0.03"/>
+            </geometry>
+            <material name="white"/>
+        </visual>
+        <collision>
+            <geometry>
+                <box size="0.3 0.15 0.03"/>
+            </geometry>
+        </collision>
+        <xacro:inertial_box mass="0.32" x="0.3" y="0.3" z="0.15">
+            <origin xyz="0 0 0" rpy="0 0 0"/>
+        </xacro:inertial_box>
+    </link>
+    <link name="back_left_wheel">
+        <visual>
+            <geometry>
+                <cylinder radius= "0.07" length="0.04"/>
+            </geometry>
+            <material name="blue"/>
+        </visual>
+        <collision>
+            <geometry>
+                <cylinder radius= "0.07" length="0.04"/>
+            </geometry>
+        </collision>
+        <xacro:inertial_cylinder mass="0.1" length="0.04" radius="0.07">
             <origin xyz="0 0 0" rpy="0 0 0"/>
         </xacro:inertial_cylinder>
     </link>
-    <gazebo reference="left_wheel">
-        <material>Gazebo/Blue</material>
-    </gazebo>
-    <!-- RIGHT WHEEL LINK -->
-    <joint name="right_wheel_joint" type="continuous">
-        <parent link="base_link"/>
-        <child link="right_wheel"/>
-        <origin xyz="0 -0.175 0" rpy="${pi/2} 0 0"/>
+    <link name="indicator_back_left_link">
+        <visual>
+            <geometry>
+                <box size="0.1 0.01 0.001"/>
+            </geometry>
+            <material name="white"/>
+        </visual>
+    </link>
+    <link name="back_right_wheel">
+        <visual>
+            <geometry>
+                <cylinder radius= "0.07" length="0.04"/>
+            </geometry>
+            <material name="blue"/>
+        </visual>
+        <collision>
+            <geometry>
+                <cylinder radius= "0.07" length="0.04"/>
+            </geometry>
+        </collision>
+        <xacro:inertial_cylinder mass="0.1" length="0.04" radius="0.07">
+            <origin xyz="0 0 0" rpy="0 0 0"/>
+        </xacro:inertial_cylinder>
+    </link>
+    <link name="indicator_back_right_link">
+        <visual>
+            <geometry>
+                <box size="0.1 0.01 0.001"/>
+            </geometry>
+            <material name="white"/>
+        </visual>
+    </link>
+    <link name="Front_left_wheel">
+        <visual>
+            <geometry>
+                <cylinder radius= "0.07" length="0.04"/>
+            </geometry>
+            <material name="blue"/>
+        </visual>
+        <collision>
+            <geometry>
+                <cylinder radius= "0.07" length="0.04"/>
+            </geometry>
+        </collision>
+        <xacro:inertial_cylinder mass="0.1" length="0.04" radius="0.07">
+            <origin xyz="0 0 0" rpy="0 0 0"/>
+        </xacro:inertial_cylinder>
+    </link>
+    <link name="Front_right_wheel">
+        <visual>
+            <geometry>
+                <cylinder radius= "0.07" length="0.04"/>
+            </geometry>
+            <material name="blue"/>
+        </visual>
+        <collision>
+            <geometry>
+                <cylinder radius= "0.07" length="0.04"/>
+            </geometry>
+        </collision>
+        <xacro:inertial_cylinder mass="0.1" length="0.04" radius="0.07">
+            <origin xyz="0 0 0" rpy="0 0 0"/>
+        </xacro:inertial_cylinder>
+    </link>
+     <link name="indicator_Front_left_link">
+        <visual>
+            <geometry>
+                <box size="0.1 0.01 0.001"/>
+            </geometry>
+            <material name="white"/>
+        </visual>
+    </link>
+    <link name="indicator_Front_right_link">
+        <visual>
+            <geometry>
+                <box size="0.1 0.01 0.001"/>
+            </geometry>
+            <material name="white"/>
+        </visual>
+    </link>
+    <link name="camera_platform_link">
+        <visual>
+            <geometry>
+                <box size="0.5 0.15 0.03"/>
+            </geometry>
+            <material name="white"/>
+        </visual>
+        <collision>
+            <geometry>
+                <box size="0.5 0.15 0.03"/>
+            </geometry>
+        </collision>
+        <xacro:inertial_box mass="0.01" x="0.3" y="0.3" z="0.15">
+            <origin xyz="0 0 0" rpy="0 0 0"/>
+        </xacro:inertial_box>
+    </link>
+    <link name="support_right">
+        <visual>
+            <geometry>
+                <box size="0.1 0.03 0.06"/>
+            </geometry>
+            <material name="white"/>
+        </visual>
+        <collision>
+            <geometry>
+                <box size="0.1 0.03 0.06"/>
+            </geometry>
+        </collision>
+        <xacro:inertial_box mass="0.5" x="0.3" y="0.3" z="0.15">
+            <origin xyz="0 0 0" rpy="0 0 0"/>
+        </xacro:inertial_box>
+    </link>
+    <link name="support_left">
+        <visual>
+            <geometry>
+                <box size="0.1 0.03 0.06"/>
+            </geometry>
+            <material name="white"/>
+        </visual>
+        <collision>
+            <geometry>
+                <box size="0.1 0.03 0.06"/>
+            </geometry>
+        </collision>
+        <xacro:inertial_box mass="0.5" x="0.3" y="0.3" z="0.15">
+            <origin xyz="0 0 0" rpy="0 0 0"/>
+        </xacro:inertial_box>
+    </link>
+    <link name="support">
+        <visual>
+            <geometry>
+                <box size="0.1 0.3 0.03"/>
+            </geometry>
+            <material name="white"/>
+        </visual>
+    </link>
+<!--================================================================ REFERENCES ================================================================================================= -->
+    <gazebo reference="base_link">
+        <material>Gazebo/White</material>
+    </gazebo>
+    <gazebo reference="Back_base_link">
+        <material>Gazebo/Blue</material>
+    </gazebo>
+    <gazebo reference="Front_base_link">
+        <material>Gazebo/Blue</material>
+    </gazebo>
+    <gazebo reference="LeftFront_wheel_support">
+        <material>Gazebo/White</material>
+    </gazebo>
+    <gazebo reference="RightFront_wheel_support">
+        <material>Gazebo/White</material>
+    </gazebo>
+    <gazebo reference="back_left_wheel">
+        <mu1>1.7</mu1>
+        <mu2>1.7</mu2>
+        <material>Gazebo/Blue</material>
+    </gazebo>
+    <gazebo reference="indicator_back_left_link">
+        <material>Gazebo/White</material>
+    </gazebo>
+    <gazebo reference="back_right_wheel">
+        <mu1>1.7</mu1>
+        <mu2>1.7</mu2>
+        <material>Gazebo/Blue</material>
+    </gazebo>
+    <gazebo reference="indicator_back_right_link">
+        <material>Gazebo/White</material>
+    </gazebo>
+    <gazebo reference="Front_left_wheel">
+        <mu1>0.1</mu1>
+        <mu2>0.1</mu2>
+        <material>Gazebo/Blue</material>
+    </gazebo>
+    <gazebo reference="indicator_Front_left_link">
+        <material>Gazebo/White</material>
+    </gazebo>
+    <gazebo reference="Front_right_wheel">
+        <mu1>0.1</mu1>
+        <mu2>0.1</mu2>
+        <material>Gazebo/Blue</material>
+    </gazebo>
+    <gazebo reference="indicator_Front_right_link">
+        <material>Gazebo/White</material>
+    </gazebo>
+    <gazebo reference="support_right">
+        <material>Gazebo/White</material>
+    </gazebo>
+    <gazebo reference="support_left">
+        <material>Gazebo/White</material>
+    </gazebo>
+<!--================================================================ JOINTS ===================================================================================================== -->
+    <joint name="reference" type="fixed">
+        <parent link="base_link"/>
+        <child link="origin"/>
+        <origin xyz="0.0 0 0.0"/>
+    </joint>
+    <joint name="Back_base_link_joint" type="fixed">
+        <parent link="base_link"/>
+        <child link="Back_base_link"/>
+        <origin xyz="-0.05 0 -0.075"/>
+    </joint>
+    <joint name="Front_base_link_joint" type="fixed">
+        <parent link="base_link"/>
+        <child link="Front_base_link"/>
+        <origin xyz="0.35 0 -0.075"/>
+    </joint>
+    <joint name="LeftFront_wheel_joint" type="fixed">
+        <parent link="base_link"/>
+        <child link="LeftFront_wheel_support"/>
+        <origin xyz="0.3 -0.135 0" rpy="-${pi/2} 0 0"/>
+    </joint>
+    <joint name="RightFront_wheel_joint" type="fixed">
+        <parent link="base_link"/>
+        <child link="RightFront_wheel_support"/>
+        <origin xyz="0.3 0.135 0" rpy="${pi/2} 0 0"/>
+    </joint>
+    <joint name="back_left_wheel_joint" type="continuous">
+        <parent link="base_link"/>
+        <child link="back_left_wheel"/>
+        <origin xyz="-0.05 -0.175 -0.075" rpy="${pi/2} 0 0"/>
         <axis xyz ="0 0 -1"/>
     </joint>
-    <link name="right_wheel">
-        <visual>
-            <geometry>
-                <cylinder radius= "0.05" length="0.04"/>
-            </geometry>
-            <material name="blue"/>
-        </visual>
-        <collision>
-            <geometry>
-                <cylinder radius= "0.05" length="0.04"/>
-            </geometry>
-        </collision>
-        <xacro:inertial_cylinder mass="0.1" length="0.04" radius="0.05">
-            <origin xyz="0 0 0" rpy="0 0 0"/>
-        </xacro:inertial_cylinder>
-    </link>
-    <gazebo reference="right_wheel">
-        <material>Gazebo/Blue</material>
-    </gazebo>
-    <!-- CASTER WHEEL LINK -->
-    <joint name="caster_wheel_joint" type="fixed">
-        <parent link="chassis"/>
-        <child link ="caster_wheel"/>
-        <origin xyz="0.24 0 0"/>
-    </joint>
-    <link name="caster_wheel">
-        <visual>
-            <geometry>
-                <sphere radius="0.05"/>
-            </geometry>
-            <material name="black"/>
-        </visual>
-        <collision>
-            <geometry>
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